File: hardware/usb-target.sch (KiCad schematic (older format))
At the start: 12 parts, among them J1 USB_A, U1 ATtiny85V-10PU

Commit message: hardware: update component value to match v-usb recommendations
Parts:
- R1: value 1K -> 1.5K
Connections:
- no-connect marks 2 -> 1
Changed lines of the file:
@@
 P 3650 3400
 F 0 "R1" V 3600 3200 50  0000 C CNN
-F 1 "1K" V 3600 3600 50  0000 C CNN
+F 1 "1.5K" V 3600 3600 50  0000 C CNN
 F 2 "Resistor_SMD:R_0805_2012Metric" V 3580 3400 50  0001 C CNN
 F 3 "~" H 3650 3400 50  0001 C CNN
@@
 $EndComp
 NoConn ~ 3350 3700
-NoConn ~ 3750 4050
 $EndSCHEMATC
